Commit message: Add files via upload

File: urdf/resetrobot.urdf (robot description, URDF)
Before this commit: robot resetrobot, 8 links, 7 joints
Links:
- added link world
Joints:
- added joint fixed: type fixed, parent world, child base_link, origin xyz=0 0 0 rpy=0 0 0
- joint last_joint: type continuous -> fixed
